File: pcbs_eagle/powersupply.sch (EAGLE design)
At the start: 0 parts

Commit message: .
Parts:
- added C1, C2: (no value), rcl:C-EU025-024X044
- added C3, C4: (no value), rcl:CPOL-EUE2,5-6E
- added D1, D2: 1N4148DO35-10, diode:1N4148DO35-10
- added IC1: 7805T, linear:7805T
- added LED1: (no value), led:LED5MM
- added R1: (no value), rcl:R-EU_0207/10
- added X1, X2, X3: JST-XH-02-PIN-LONG-PAD, Rembrandt Electronics - JST XH Connectors v1-0:JST-XH-02-PIN-LONG-PAD
Connections:
- new net GND: C1.2, C2.1, C3.-, C4.-, IC1.GND, LED1.C, X1-2.S, X2-1.S, X3-1.S
- new net N$1: D1.A, X1-1.S, X3-2.S
- new net N$2: C1.1, C3.+, D1.C, D2.C, IC1.VI
- new net N$4: C2.2, C4.+, D2.A, IC1.VO, R1.1, X2-2.S
- new net N$6: LED1.A, R1.2
